File: electronics/PowerManagement.kicad_sch (KiCad schematic)
At the start: 35 parts, among them J1 Jumper, J6 Battery Port, J6 Button11, J6 Button12, J6 Button21, J6 Button22, J6 Button31, J6 Button32, Q1 BC547, U2 AMS1117-3.3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

Commit message: Improve readme & rename files
Parts:
- renumbered C10 to C?, C7 to C?, D2 to D?, J6 to J?, J1 to J?, U2 to U?
