File: electronics/GarageRemote.kicad_pcb (KiCad board)
At the start: 2 copper layers, 36.1 x 31.2 mm, 27 parts, among them J1 Battery, J10 Button32, J2 CC1101 Module, J3 ICSP, J4 Button21, J5 Button31, J7 Button11, J8 Button12, J9 Button22, U1 AMS1117-3.3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

Commit message: Fix ground plane
Connections:
- U2 pad 12: CSN_CC1101 -> unconnected-(U2-PB0-Pad12)
- U2 pad 13: RF_DATA0 -> unconnected-(U2-PB1-Pad13)
- U2 pad 14: RF_DATA2 -> unconnected-(U2-PB2-Pad14)
- U2 pad 24: unconnected-(U2-PC1-Pad24) -> CSN_CC1101
- U2 pad 25: unconnected-(U2-PC2-Pad25) -> RF_DATA0
- U2 pad 26: unconnected-(U2-PC3-Pad26) -> RF_DATA2
Routing:
- net GND: track 120.2 -> 0.00 mm, vias 1 -> 2
- net CSN_CC1101: track 3.68 -> 65.1 mm, vias 0 -> 1
- net RF_DATA2: track 6.77 -> 48.3 mm, vias 0 -> 1
- net RF_DATA0: track 6.14 -> 24.9 mm
- net B32: track 27.8 -> 41.5 mm, vias 2 -> 0
- net RESET: track 34.3 -> 45.3 mm
- net B31: track 37.9 -> 48.0 mm
- net +3.3V: track 94.0 -> 85.0 mm, vias 1 -> 3
- net VBAT-: track 80.6 -> 71.7 mm
- net Net-(D11-K): track 41.5 -> 34.9 mm
- net Net-(D5-K): track 27.9 -> 25.5 mm
- net Net-(D10-K): track 33.7 -> 36.0 mm
- net B11: track 26.0 -> 27.8 mm, vias 0 -> 2
- net B21: track 29.8 -> 31.6 mm
- net SCK: track 31.4 -> 29.7 mm
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- added copper zone on B.Cu, net GND
- added copper zone on F.Cu, net GND
- removed copper zone on B.Cu, net (none)
- removed copper zone on F.Cu, net (none)
