File: electronics/GarageRemote.kicad_sch (KiCad schematic)
At the start: 47 parts, among them J1 CC1101 Module, J10 Button32, J11 Battery Port, J2 SERIAL, J3 ICSP, J4 Button21, J5 Button31, J6 Button11, J8 Button12, J9 Button22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

Commit message: Finished 1.1.0 design
Parts:
- removed C1, C2: 22pF, Capacitor_SMD:C_0805_2012Metric_Pad1.18x1.45mm_HandSolder, symbol Device:C_Small
- removed J2: SERIAL, Connector_PinHeader_2.54mm:PinHeader_1x04_P2.54mm_Vertical, symbol Connector:Conn_01x04_Pin
- removed Y1: 16MHz, Crystal:Crystal_HC49-4H_Vertical, symbol Device:Crystal_Small
- J10, J4, J5, J6, J8, J9: footprint AA_Footprints:4.5mm switch -> AA_Footprints:ButtonSMD 6x6
Other:
- moved on the sheet: J3
